Commit message: all servers tested

File: ur16e_dual_arm_description/urdf/dual_arm.urdf (robot description, URDF)
Before this commit: robot dual_arm_ur16e, 27 links, 26 joints
Links:
- link left_suction_gripper: geometry collision cylinder length=0.22 radius=0.05; visual cylinder length=0.22 radius=0.05
- link right_rws_gripper: geometry collision cylinder length=0.14 radius=0.05; visual cylinder length=0.14 radius=0.05
Joints:
- joint left_suction_gripper-poi: origin xyz=0 0 0.05 rpy=0 0 0 -> xyz=0 0 0.11 rpy=0 0 0
- joint left_wrist_3_link-suction_gripper: origin xyz=0 0 0.05 rpy=0 0 0 -> xyz=0 0 0.11 rpy=0 0 0
- joint right_rws_gripper-poi: origin xyz=0 0 0.05 rpy=0 0 0 -> xyz=0 0 0.07 rpy=0 0 0
- joint right_wrist_3_link-_rws_gripper: origin xyz=0 0 0.05 rpy=0 0 0 -> xyz=0 0 0.07 rpy=0 0 0
